File: Hardware/Frontend/Frontend.sch (KiCad schematic (older format))
At the start: 43 parts, among them J1 power, J2 Conn_Coaxial, J3 Conn_Coaxial, U1 OPA333xxD, U2 OPA333xxD, U4 LM358_DFN

Commit message: update schematic, create pcupdate schematic, create pcbb update schematic, create pcupdate schematic, create pcbb# Please enter the commit message for your changes. Lines starting
Parts:
- removed BT1, BT2, BT3, BT4: 12V, SemiconductorRadioactivityDetector:A23Single, symbol Device:Battery_Cell
- removed C1: 1u/16V, Capacitors_Tantalum_SMD:CP_Tantalum_Case-A_EIA-3216-18_Hand, symbol Device:CP
- removed C10: 4p7+2p2, Capacitors_SMD:C_0805_HandSoldering, symbol Device:C
- removed C11, C2, C3, C4, C5, C8, C9: 100n, Capacitors_SMD:C_0805_HandSoldering, symbol Device:C
- removed C12: solder bridge, Capacitors_SMD:C_0805_HandSoldering, symbol Device:C
- removed C6: 2p2, Capacitors_SMD:C_0805_HandSoldering, symbol Device:C
- removed C7: 1n, Capacitors_SMD:C_0805_HandSoldering, symbol Device:C
- removed D1, D2, D3: BPW34, Diodes_THT:D_DO-35_SOD27_P5.08mm_Vertical_KathodeUp, symbol Device:D_Photo
- removed H1, H2, H3: MountingHole_Pad, Mounting_Holes:MountingHole_3.5mm_Pad, symbol Mechanical:MountingHole_Pad
- removed J1: power, Connector_PinHeader_2.54mm:PinHeader_1x02_P2.54mm_Vertical, symbol Connector:Conn_01x02_Male
- removed J2, J3: Conn_Coaxial, Connectors:BNC, symbol Connector:Conn_Coaxial
- removed L1: u68, Inductors_SMD:L_1812, symbol Device:L_Core_Ferrite
- removed R1, R10, R11, R12, R2, R5, R7: 10k, Resistors_SMD:R_0805_HandSoldering, symbol Device:R
- removed R13, R9: not mounted, Resistors_SMD:R_0805_HandSoldering, symbol Device:R
- removed R3: 0R, Resistors_SMD:R_0805_HandSoldering, symbol Device:R
- removed R4: 10G, Resistors_SMD:R_0805_HandSoldering, symbol Device:R
- removed R6: 10k, Resistors_THT:R_Axial_DIN0207_L6.3mm_D2.5mm_P10.16mm_Horizontal, symbol Device:R
- removed R8: 10M, Resistors_SMD:R_0805_HandSoldering, symbol Device:R
- removed RV1: 100k, Potentiometers:Potentiometer_Trimmer_Bourns_3296W, symbol Device:R_POT_TRIM
- removed U1, U2: OPA333xxD, Housings_SOIC:SOIC-8_3.9x4.9mm_Pitch1.27mm, symbol Amplifier_Operational:OPA333xxD
- removed U4: LM358_DFN, Housings_SOIC:SOIC-8_3.9x4.9mm_Pitch1.27mm, symbol Amplifier_Operational:LM358_DFN
