File: Hardware/Detector/Detector2.kicad_sch (KiCad schematic)
At the start: 27 parts, among them J4 Conn_Coaxial, U4 OPA145ID, U5 OPA145ID, U6 OPA145ID

Commit message: switch to low cost solution
Parts:
- removed C11, C12, C13, C14, C17, C18, C20: 100n, Capacitor_SMD:C_0402_1005Metric, symbol Device:C
- removed C15: 2p2, Capacitor_SMD:C_0402_1005Metric, symbol Device:C
- removed C16: 1n, Capacitor_SMD:C_0402_1005Metric, symbol Device:C
- removed C19: 4p7+2p2, Capacitor_SMD:C_0402_1005Metric, symbol Device:C
- removed D3: BPW34, LED_THT:LED_Rectangular_W5.0mm_H5.0mm, symbol Device:D_Photo
- removed J4: Conn_Coaxial, Connector_Coaxial:SMA_Molex_73251-2200_Horizontal, symbol Connector:Conn_Coaxial
- removed L2: u68, Inductor_SMD:L_0805_2012Metric, symbol Device:L_Core_Ferrite
- removed R13, R14, R17, R18, R19, R21, R23: 10k, Resistor_SMD:R_0402_1005Metric, symbol Device:R
- removed R16: 10G, Resistor_SMD:R_0805_2012Metric, symbol Device:R
- removed R20: 10M, Resistor_SMD:R_0402_1005Metric, symbol Device:R
- removed R22: 0R, Resistor_SMD:R_0402_1005Metric, symbol Device:R
- removed R24: not mounted, Resistor_SMD:R_0402_1005Metric, symbol Device:R
- removed U4, U5, U6: OPA145ID, Package_SO:SOIC-8_3.9x4.9mm_P1.27mm, symbol OPA145ID:OPA145ID
