File: Hardware/Detector/Detector3.kicad_sch (KiCad schematic)
At the start: 27 parts, among them J5 Conn_Coaxial, U7 OPA145ID, U8 OPA145ID, U9 OPA145ID

Commit message: switch to low cost solution
Parts:
- removed C21, C22, C23, C24, C27, C28, C30: 100n, Capacitor_SMD:C_0402_1005Metric, symbol Device:C
- removed C25: 2p2, Capacitor_SMD:C_0402_1005Metric, symbol Device:C
- removed C26: 1n, Capacitor_SMD:C_0402_1005Metric, symbol Device:C
- removed C29: 4p7+2p2, Capacitor_SMD:C_0402_1005Metric, symbol Device:C
- removed D5: BPW34, LED_THT:LED_Rectangular_W5.0mm_H5.0mm, symbol Device:D_Photo
- removed J5: Conn_Coaxial, Connector_Coaxial:SMA_Molex_73251-2200_Horizontal, symbol Connector:Conn_Coaxial
- removed L3: u68, Inductor_SMD:L_0805_2012Metric, symbol Device:L_Core_Ferrite
- removed R25, R26, R29, R30, R31, R33, R35: 10k, Resistor_SMD:R_0402_1005Metric, symbol Device:R
- removed R28: 10G, Resistor_SMD:R_0805_2012Metric, symbol Device:R
- removed R32: 10M, Resistor_SMD:R_0402_1005Metric, symbol Device:R
- removed R34: 0R, Resistor_SMD:R_0402_1005Metric, symbol Device:R
- removed R36: not mounted, Resistor_SMD:R_0402_1005Metric, symbol Device:R
- removed U7, U8, U9: OPA145ID, Package_SO:SOIC-8_3.9x4.9mm_P1.27mm, symbol OPA145ID:OPA145ID
