File: Hardware/Detector/Detector4.kicad_sch (KiCad schematic)
At the start: 27 parts, among them J6 Conn_Coaxial, U10 OPA145ID, U11 OPA145ID, U12 OPA145ID

Commit message: switch to low cost solution
Parts:
- removed C31, C32, C33, C34, C37, C38, C40: 100n, Capacitor_SMD:C_0402_1005Metric, symbol Device:C
- removed C35: 2p2, Capacitor_SMD:C_0402_1005Metric, symbol Device:C
- removed C36: 1n, Capacitor_SMD:C_0402_1005Metric, symbol Device:C
- removed C39: 4p7+2p2, Capacitor_SMD:C_0402_1005Metric, symbol Device:C
- removed D7: BPW34, LED_THT:LED_Rectangular_W5.0mm_H5.0mm, symbol Device:D_Photo
- removed J6: Conn_Coaxial, Connector_Coaxial:SMA_Molex_73251-2200_Horizontal, symbol Connector:Conn_Coaxial
- removed L4: u68, Inductor_SMD:L_0805_2012Metric, symbol Device:L_Core_Ferrite
- removed R37, R38, R41, R42, R43, R45, R47: 10k, Resistor_SMD:R_0402_1005Metric, symbol Device:R
- removed R40: 10G, Resistor_SMD:R_0805_2012Metric, symbol Device:R
- removed R44: 10M, Resistor_SMD:R_0402_1005Metric, symbol Device:R
- removed R46: 0R, Resistor_SMD:R_0402_1005Metric, symbol Device:R
- removed R48: not mounted, Resistor_SMD:R_0402_1005Metric, symbol Device:R
- removed U10, U11, U12: OPA145ID, Package_SO:SOIC-8_3.9x4.9mm_P1.27mm, symbol OPA145ID:OPA145ID
