File: Hardware/Detector/Detector5.kicad_sch (KiCad schematic)
At the start: 27 parts, among them J7 Conn_Coaxial, U13 OPA145ID, U14 OPA145ID, U15 OPA145ID

Commit message: switch to low cost solution
Parts:
- removed C41, C42, C43, C44, C47, C48, C50: 100n, Capacitor_SMD:C_0402_1005Metric, symbol Device:C
- removed C45: 2p2, Capacitor_SMD:C_0402_1005Metric, symbol Device:C
- removed C46: 1n, Capacitor_SMD:C_0402_1005Metric, symbol Device:C
- removed C49: 4p7+2p2, Capacitor_SMD:C_0402_1005Metric, symbol Device:C
- removed D9: BPW34, LED_THT:LED_Rectangular_W5.0mm_H5.0mm, symbol Device:D_Photo
- removed J7: Conn_Coaxial, Connector_Coaxial:SMA_Molex_73251-2200_Horizontal, symbol Connector:Conn_Coaxial
- removed L5: u68, Inductor_SMD:L_0805_2012Metric, symbol Device:L_Core_Ferrite
- removed R49, R50, R53, R54, R55, R57, R59: 10k, Resistor_SMD:R_0402_1005Metric, symbol Device:R
- removed R52: 10G, Resistor_SMD:R_0805_2012Metric, symbol Device:R
- removed R56: 10M, Resistor_SMD:R_0402_1005Metric, symbol Device:R
- removed R58: 0R, Resistor_SMD:R_0402_1005Metric, symbol Device:R
- removed R60: not mounted, Resistor_SMD:R_0402_1005Metric, symbol Device:R
- removed U13, U14, U15: OPA145ID, Package_SO:SOIC-8_3.9x4.9mm_P1.27mm, symbol OPA145ID:OPA145ID
